File: m232.brd (EAGLE design)
At the start: 40 x 40 mm, 35 parts, among them CN1 DIP-BLACK-FEMALE-HEADER-VERT(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

Commit message: Add files via upload
Parts:
- U1, U2, U3: value (none) -> MAX3232
Connections:
- removed net VCC: J1.3
Routing:
- net GND: track 453.5 -> 447.8 mm, vias 36 -> 33
Other:
- board text added: "0.1" * 8P"
