File: m232.sch (EAGLE design)
At the start: 35 parts, among them CN1 DIP-BLACK-FEMALE-HEADER-VERT(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

Commit message: Add files via upload
Parts:
- U1, U2, U3: value (none) -> MAX3232
Connections:
- removed net VCC: J1.3
Other:
- moved on the sheet: CN1, J1
